Commit message: Add WEC HIL dynamometer setup: register PTO motor (axis1) in ros2_control
- URDF: rename robot to odrive_wec_dyno, add pto_link/pto_joint, register
  pto_joint (node_id=1) inside the existing ODriveSystem hardware block
- controllers.yaml: add pto_effort_controller for pto_joint
- odrive_velocity_pid/controllers.yaml: add pto_effort_controller
- launch: add pto_controller_spawner node
- READMEs: document WEC HIL dyno concept, Phase 1 passive damping via
  odrivetool, oscilloscope power measurement, Phase 2 roadmap

Co-authored-by: salhus <84348506+salhus@users.noreply.github.com>
Agent-Logs-Url: https://github.com/salhus/hil_odrive_ros2_control/sessions/644bc690-b421-4ec5-8bdf-9eb185c49550

File: src/hil_odrive_ros2_control/description/urdf/motor.urdf.xacro (robot description, xacro)
@@ -1,4 +1,4 @@
 <?xml version="1.0"?>
-<robot xmlns:xacro="http://www.ros.org/wiki/xacro" name="odrive_single_motor">
+<robot xmlns:xacro="http://www.ros.org/wiki/xacro" name="odrive_wec_dyno">
   <!-- Minimal kinematic tree -->
   <link name="base_link"/>
@@ -10,5 +10,13 @@
     <axis xyz="0 0 1"/>
   </joint>
-  <!-- ros2_control hardware -->
+  <!-- PTO motor (axis1) — same shaft as motor_joint, passive linear damper -->
+  <link name="pto_link"/>
+  <joint name="pto_joint" type="continuous">
+    <parent link="motor_link"/>
+    <child link="pto_link"/>
+    <origin xyz="0 0 0" rpy="0 0 0"/>
+    <axis xyz="0 0 1"/>
+  </joint>
+  <!-- ros2_control hardware — both axes on the same ODrive board / CAN bus -->
   <ros2_control name="ODriveSystem" type="system">
     <hardware>
@@ -17,5 +25,5 @@
       <param name="can">can0</param>
     </hardware>
-    <!-- Single joint mapping to ODrive node_id -->
+    <!-- Motor 1: Hydro Emulator (ODrive axis0, node_id=0) -->
     <joint name="motor_joint">
       <param name="node_id">0</param>
@@ -29,4 +37,16 @@
       <state_interface name="position"/>
     </joint>
+    <!-- Motor 2: PTO / Power Take-Off (ODrive axis1, node_id=1) -->
+    <joint name="pto_joint">
+      <param name="node_id">1</param>
+      <!-- Command interfaces the hardware plugin exports -->
+      <command_interface name="effort"/>
+      <command_interface name="velocity"/>
+      <command_interface name="position"/>
+      <!-- State interfaces the hardware plugin exports -->
+      <state_interface name="effort"/>
+      <state_interface name="velocity"/>
+      <state_interface name="position"/>
+    </joint>
   </ros2_control>
 </robot>
